Commit message: absolute mesh path (now loaded in rviz)

File: resources/centauro/urdf/centauro_horizon.urdf (robot description, URDF)
Before this commit: robot centauro, 97 links, 96 joints
Links:
- link ankle1_1: geometry collision mesh filename=/home/idadiotis/ocs2_ws/src/ocs2_robotic_assets/resources/c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 scale=0.001 0.001 -0.001; visual mesh filename=package://centauro_urdf/meshes/v2/ankle-pitch.stl scale=0.001 0.001 -0.001
- link ankle1_2: geometry collision mesh filename=/home/idadiotis/ocs2_ws/src/ocs2_robotic_assets/resources/c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 scale=0.001 0.001 0.001; visual mesh filename=package://centauro_urdf/meshes/v2/ankle-pitch.stl scale=0.001 0.001 0.001
- link ankle1_3: geometry collision mesh filename=/home/idadiotis/ocs2_ws/src/ocs2_robotic_assets/resources/c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 scale=0.001 0.001 -0.001; visual mesh filename=package://centauro_urdf/meshes/v2/ankle-pitch.stl scale=0.001 0.001 -0.001
- link ankle1_4: geometry collision mesh filename=/home/idadiotis/ocs2_ws/src/ocs2_robotic_assets/resources/c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 scale=0.001 0.001 0.001; visual mesh filename=package://centauro_urdf/meshes/v2/ankle-pitch.stl scale=0.001 0.001 0.001
- link ankle2_1: geometry collision mesh filename=/home/idadiotis/ocs2_ws/src/ocs2_robotic_assets/resources/c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 scale=0.001 -0.001 0.001; visual mesh filename=package://centauro_urdf/meshes/v2/ankle-yaw.stl scale=0.001 -0.001 0.001
- link ankle2_2: geometry collision mesh filename=/home/idadiotis/ocs2_ws/src/ocs2_robotic_assets/resources/c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 scale=0.001 0.001 0.001; visual mesh filename=package://centauro_urdf/meshes/v2/ankle-yaw.stl scale=0.001 0.001 0.001
- link ankle2_3: geometry collision mesh filename=/home/idadiotis/ocs2_ws/src/ocs2_robotic_assets/resources/c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 scale=0.001 -0.001 0.001; visual mesh filename=package://centauro_urdf/meshes/v2/ankle-yaw.stl scale=0.001 -0.001 0.001
- link ankle2_4: geometry collision mesh filename=/home/idadiotis/ocs2_ws/src/ocs2_robotic_assets/resources/c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 scale=0.001 0.001 0.001; visual mesh filename=package://centauro_urdf/meshes/v2/ankle-yaw.stl scale=0.001 0.001 0.001
- link arm1_1: geometry collision mesh filename=/home/idadiotis/ocs2_ws/src/ocs2_robotic_assets/resources/c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 scale=0.001 -0.001 0.001; visual mesh filename=package://centauro_urdf/meshes/ShoulderPitch.STL scale=0.001 -0.001 0.001
- link arm1_2: geometry collision mesh filename=/home/idadiotis/ocs2_ws/src/ocs2_robotic_assets/resources/c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 scale=0.001 -0.001 0.001; visual mesh filename=package://centauro_urdf/meshes/ShoulderRoll.STL scale=0.001 -0.001 0.001
- link arm1_3: geometry collision mesh filename=/home/idadiotis/ocs2_ws/src/ocs2_robotic_assets/resources/c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 scale=0.001 -0.001 0.001; visual mesh filename=package://centauro_urdf/meshes/ShoulderYaw.STL scale=0.001 -0.001 0.001
- link arm1_4: geometry collision mesh filename=/home/idadiotis/ocs2_ws/src/ocs2_robotic_assets/resources/c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 scale=0.001 -0.001 0.001; visual mesh filename=package://centauro_urdf/meshes/Elbow.STL scale=0.001 -0.001 0.001
- link arm1_5: geometry collision mesh filename=/home/idadiotis/ocs2_ws/src/ocs2_robotic_assets/resources/c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 scale=0.001 -0.001 0.001; visual mesh filename=package://centauro_urdf/meshes/Forearm.STL scale=0.001 -0.001 0.001
- link arm1_6: geometry collision mesh filename=/home/idadiotis/ocs2_ws/src/ocs2_robotic_assets/resources/c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 scale=0.001 -0.001 0.001; visual mesh filename=package://centauro_urdf/meshes/ForearmPitch.STL scale=0.001 -0.001 0.001
- link arm1_7: geometry collision mesh filename=/home/idadiotis/ocs2_ws/src/ocs2_robotic_assets/resources/c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 scale=0.001 -0.001 0.001; visual mesh filename=package://centauro_urdf/meshes/ForearmYaw.STL scale=0.001 -0.001 0.001
- link arm2_1: geometry collision mesh filename=/home/idadiotis/ocs2_ws/src/ocs2_robotic_assets/resources/c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 scale=0.001 0.001 0.001; visual mesh filename=package://centauro_urdf/meshes/ShoulderPitch.STL scale=0.001 0.001 0.001
- link arm2_2: geometry collision mesh filename=/home/idadiotis/ocs2_ws/src/ocs2_robotic_assets/resources/c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 scale=0.001 0.001 0.001; visual mesh filename=package://centauro_urdf/meshes/ShoulderRoll.STL scale=0.001 0.001 0.001
- link arm2_3: geometry collision mesh filename=/home/idadiotis/ocs2_ws/src/ocs2_robotic_assets/resources/c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 scale=0.001 0.001 0.001; visual mesh filename=package://centauro_urdf/meshes/ShoulderYaw.STL scale=0.001 0.001 0.001
- link arm2_4: geometry collision mesh filename=/home/idadiotis/ocs2_ws/src/ocs2_robotic_assets/resources/c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 scale=0.001 0.001 0.001; visual mesh filename=package://centauro_urdf/meshes/Elbow.STL scale=0.001 0.001 0.001
- link arm2_5: geometry collision mesh filename=/home/idadiotis/ocs2_ws/src/ocs2_robotic_assets/resources/c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 scale=0.001 0.001 0.001; visual mesh filename=package://centauro_urdf/meshes/Forearm.STL scale=0.001 0.001 0.001
- link arm2_6: geometry collision mesh filename=/home/idadiotis/ocs2_ws/src/ocs2_robotic_assets/resources/c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 scale=0.001 0.001 0.001; visual mesh filename=package://centauro_urdf/meshes/ForearmPitch.STL scale=0.001 0.001 0.001
- link arm2_7: geometry collision mesh filename=/home/idadiotis/ocs2_ws/src/ocs2_robotic_assets/resources/c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 scale=0.001 0.001 0.001; visual mesh filename=package://centauro_urdf/meshes/ForearmYaw.STL scale=0.001 0.001 0.001
- link ball1: geometry collision mesh filename=/home/idadiotis/ocs2_ws/src/ocs2_robotic_assets/resources/c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 scale=0.001 0.001 0.001; visual mesh filename=package://centauro_urdf/meshes/BallHand.stl scale=0.001 0.001 0.001
- link ball2: geometry collision mesh filename=/home/idadiotis/ocs2_ws/src/ocs2_robotic_assets/resources/c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 scale=0.001 0.001 0.001; visual mesh filename=package://centauro_urdf/meshes/BallHand.stl scale=0.001 0.001 0.001
- link base_link: geometry collision mesh filename=/home/idadiotis/ocs2_ws/src/ocs2_robotic_assets/resources/c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 scale=0.001 0.001 0.001; visual mesh filename=package://centauro_urdf/meshes/v2/pelvis.stl scale=0.001 0.001 0.001
- link d435_head_motor: geometry collision mesh filename=/home/idadiotis/ocs2_ws/src/ocs2_robotic_assets/resources/c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 scale=0.001 0.001 0.001; visual mesh filename=package://centauro_urdf/meshes/neck-pitch_mesh.stl scale=0.001 0.001 0.001
- link hip1_1: geometry collision mesh filename=/home/idadiotis/ocs2_ws/src/ocs2_robotic_assets/resources/c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 scale=0.001 -0.001 0.001; visual mesh filename=package://centauro_urdf/meshes/v2/hip-yaw.stl scale=0.001 -0.001 0.001
- link hip1_2: geometry collision mesh filename=/home/idadiotis/ocs2_ws/src/ocs2_robotic_assets/resources/c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 scale=0.001 0.001 0.001; visual mesh filename=package://centauro_urdf/meshes/v2/hip-yaw.stl scale=0.001 0.001 0.001
- link hip1_3: geometry collision mesh filename=/home/idadiotis/ocs2_ws/src/ocs2_robotic_assets/resources/c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 scale=0.001 -0.001 0.001; visual mesh filename=package://centauro_urdf/meshes/v2/hip-yaw.stl scale=0.001 -0.001 0.001
- link hip1_4: geometry collision mesh filename=/home/idadiotis/ocs2_ws/src/ocs2_robotic_assets/resources/c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 scale=0.001 0.001 0.001; visual mesh filename=package://centauro_urdf/meshes/v2/hip-yaw.stl scale=0.001 0.001 0.001
- link hip2_1: geometry collision mesh filename=/home/idadiotis/ocs2_ws/src/ocs2_robotic_assets/resources/c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 scale=0.001 0.001 -0.001; visual mesh filename=package://centauro_urdf/meshes/v2/hip-pitch.stl scale=0.001 0.001 -0.001
- link hip2_2: geometry collision mesh filename=/home/idadiotis/ocs2_ws/src/ocs2_robotic_assets/resources/c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 scale=0.001 0.001 0.001; visual mesh filename=package://centauro_urdf/meshes/v2/hip-pitch.stl scale=0.001 0.001 0.001
- link hip2_3: geometry collision mesh filename=/home/idadiotis/ocs2_ws/src/ocs2_robotic_assets/resources/c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 scale=0.001 0.001 -0.001; visual mesh filename=package://centauro_urdf/meshes/v2/hip-pitch.stl scale=0.001 0.001 -0.001
- link hip2_4: geometry collision mesh filename=/home/idadiotis/ocs2_ws/src/ocs2_robotic_assets/resources/c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 scale=0.001 0.001 0.001; visual mesh filename=package://centauro_urdf/meshes/v2/hip-pitch.stl scale=0.001 0.001 0.001
- link knee_1: geometry collision mesh filename=/home/idadiotis/ocs2_ws/src/ocs2_robotic_assets/resources/c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 scale=0.001 0.001 -0.001; visual mesh filename=package://centauro_urdf/meshes/v2/knee.stl scale=0.001 0.001 -0.001
- link knee_2: geometry collision mesh filename=/home/idadiotis/ocs2_ws/src/ocs2_robotic_assets/resources/c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 scale=0.001 0.001 0.001; visual mesh filename=package://centauro_urdf/meshes/v2/knee.stl scale=0.001 0.001 0.001
- link knee_3: geometry collision mesh filename=/home/idadiotis/ocs2_ws/src/ocs2_robotic_assets/resources/c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 scale=0.001 0.001 -0.001; visual mesh filename=package://centauro_urdf/meshes/v2/knee.stl scale=0.001 0.001 -0.001
- link knee_4: geometry collision mesh filename=/home/idadiotis/ocs2_ws/src/ocs2_robotic_assets/resources/c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 scale=0.001 0.001 0.001; visual mesh filename=package://centauro_urdf/meshes/v2/knee.stl scale=0.001 0.001 0.001
- link neck_1: geometry collision mesh filename=/home/idadiotis/ocs2_ws/src/ocs2_robotic_assets/resources/c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 scale=0.001 0.001 0.001; visual mesh filename=package://centauro_urdf/meshes/head-base_mesh.stl scale=0.001 0.001 0.001
- link torso_2: geometry collision mesh filename=/home/idadiotis/ocs2_ws/src/ocs2_robotic_assets/resources/c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 scale=0.001 0.001 0.001; visual mesh filename=package://centauro_urdf/meshes/link1_no_head.stl scale=0.001 0.001 0.001
- link velodyne_motor: geometry collision mesh filename=/home/idadiotis/ocs2_ws/src/ocs2_robotic_assets/resources/c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 scale=0.001 0.001 0.001; visual mesh filename=package://centauro_urdf/meshes/lidar_mesh.stl scale=0.001 0.001 0.001

Commit message: replace meshes with capsules

File: resources/centauro/urdf/centauro_horizon.urdf (robot description, URDF)
Before this commit: robot centauro, 97 links, 96 joints
Links:
- link T265_camera_pose_frame: geometry collision cylinder length=0.1022528557886848 radius=0.0142751; collision sphere radius=0.0142751
- link ankle1_1: geometry collision cylinder length=0.049256315666076876 radius=0.0792379; collision sphere radius=0.0792379
- link ankle1_2: geometry collision cylinder length=0.047884051265172006 radius=0.0781037; collision sphere radius=0.0781037
- link ankle1_3: geometry collision cylinder length=0.049256315666076876 radius=0.0792379; collision sphere radius=0.0792379
- link ankle1_4: geometry collision cylinder length=0.047884051265172006 radius=0.0781037; collision sphere radius=0.0781037
- link ankle2_1: geometry collision cylinder length=0.07370263129636398 radius=0.0813545; collision sphere radius=0.0813545
- link ankle2_2: geometry collision cylinder length=0.07370263129636398 radius=0.0813545; collision sphere radius=0.0813545
- link ankle2_3: geometry collision cylinder length=0.07370263129636398 radius=0.0813545; collision sphere radius=0.0813545
- link ankle2_4: geometry collision cylinder length=0.07370263129636398 radius=0.0813545; collision sphere radius=0.0813545
- link arm1_1: geometry collision cylinder length=0.03739768494560427 radius=0.0698859; collision sphere radius=0.0698859
- link arm1_2: geometry collision cylinder length=0.12799269981445732 radius=0.0700645; collision sphere radius=0.0700645
- link arm1_3: geometry collision cylinder length=0.06082252644344949 radius=0.0896121; collision sphere radius=0.0896121
- link arm1_4: geometry collision cylinder length=0.08713418572944408 radius=0.0600429; collision sphere radius=0.0600429
- link arm1_5: geometry collision cylinder length=0.08434739747702548 radius=0.0804108; collision sphere radius=0.0804108
- link arm1_6: geometry collision cylinder length=0.11425141871384588 radius=0.0583263; collision sphere radius=0.0583263
- link arm1_7: geometry collision cylinder length=0.009167307493588288 radius=0.0207073; collision sphere radius=0.0207073
- link arm2_1: geometry collision cylinder length=0.03739768494560427 radius=0.0698859; collision sphere radius=0.0698859
- link arm2_2: geometry collision cylinder length=0.12799269981445732 radius=0.0700645; collision sphere radius=0.0700645
- link arm2_3: geometry collision cylinder length=0.06082252644344949 radius=0.0896121; collision sphere radius=0.0896121
- link arm2_4: geometry collision cylinder length=0.08713418572944408 radius=0.0600429; collision sphere radius=0.0600429
- link arm2_5: geometry collision cylinder length=0.08434739747702548 radius=0.0804108; collision sphere radius=0.0804108
- link arm2_6: geometry collision cylinder length=0.11425141871384588 radius=0.0583263; collision sphere radius=0.0583263
- link arm2_7: geometry collision cylinder length=0.009167307493588288 radius=0.0207073; collision sphere radius=0.0207073
- link ball1: geometry collision cylinder length=9.940076835940455e-05 radius=0.0709883; collision sphere radius=0.0709883
- link ball2: geometry collision cylinder length=9.940076835940455e-05 radius=0.0709883; collision sphere radius=0.0709883
- link base_link: geometry collision cylinder length=0.38594139791384763 radius=0.213204; collision sphere radius=0.213204
- link d435_head_motor: geometry collision cylinder length=0.12134423548428976 radius=0.0261699; collision sphere radius=0.0261699
- link hip1_1: geometry collision cylinder length=0.03069545889898954 radius=0.0747223; collision sphere radius=0.0747223
- link hip1_2: geometry collision cylinder length=0.03069545889898954 radius=0.0747223; collision sphere radius=0.0747223
- link hip1_3: geometry collision cylinder length=0.03069545889898954 radius=0.0747223; collision sphere radius=0.0747223
- link hip1_4: geometry collision cylinder length=0.03069545889898954 radius=0.0747223; collision sphere radius=0.0747223
- link hip2_1: geometry collision cylinder length=0.2919804521727749 radius=0.0808941; collision sphere radius=0.0808941
- link hip2_2: geometry collision cylinder length=0.2919804521727749 radius=0.0808941; collision sphere radius=0.0808941
- link hip2_3: geometry collision cylinder length=0.2919804521727749 radius=0.0808941; collision sphere radius=0.0808941
- link hip2_4: geometry collision cylinder length=0.2919804521727749 radius=0.0808941; collision sphere radius=0.0808941
- link knee_1: geometry collision cylinder length=0.19275022460612404 radius=0.0664305; collision sphere radius=0.0664305
- link knee_2: geometry collision cylinder length=0.19275022460612404 radius=0.0664305; collision sphere radius=0.0664305
- link knee_3: geometry collision cylinder length=0.19275022460612404 radius=0.0664305; collision sphere radius=0.0664305
- link knee_4: geometry collision cylinder length=0.19275022460612404 radius=0.0664305; collision sphere radius=0.0664305
- link neck_1: geometry collision cylinder length=0.16454098025546557 radius=0.100414; collision sphere radius=0.100414
- link torso_2: geometry collision cylinder length=0.09543675990850982 radius=0.158224; collision sphere radius=0.158224
- link velodyne_calib_base_link: geometry collision cylinder length=0.0717 radius=0.0516; collision sphere radius=0.0516
- link velodyne_motor: geometry collision cylinder length=0.032463112134515464 radius=0.0544637; collision sphere radius=0.0544637
- link wheel_1: geometry collision cylinder length=0.11 radius=0.078; collision sphere radius=0.078
- link wheel_2: geometry collision cylinder length=0.11 radius=0.078; collision sphere radius=0.078
- link wheel_3: geometry collision cylinder length=0.11 radius=0.078; collision sphere radius=0.078
- link wheel_4: geometry collision cylinder length=0.11 radius=0.078; collision sphere radius=0.078
