Commit message: capsules were implemented with multiple collision objects so for now removed the spheres. next step is to add <collision_checking> tags

File: resources/centauro/urdf/centauro_horizon.urdf (robot description, URDF)
Before this commit: robot centauro, 97 links, 96 joints
Links:
- link T265_camera_pose_frame: geometry collision cylinder length=0.1022528557886848 radius=0.0142751; visual mesh filename=package://realsense_gazebo_description/meshes/t265_full.stl scale=0.001 0.001 0.001
- link ankle1_1: geometry collision cylinder length=0.049256315666076876 radius=0.0792379; visual mesh filename=package://centauro_urdf/meshes/v2/ankle-pitch.stl scale=0.001 0.001 -0.001
- link ankle1_2: geometry collision cylinder length=0.047884051265172006 radius=0.0781037; visual mesh filename=package://centauro_urdf/meshes/v2/ankle-pitch.stl scale=0.001 0.001 0.001
- link ankle1_3: geometry collision cylinder length=0.049256315666076876 radius=0.0792379; visual mesh filename=package://centauro_urdf/meshes/v2/ankle-pitch.stl scale=0.001 0.001 -0.001
- link ankle1_4: geometry collision cylinder length=0.047884051265172006 radius=0.0781037; visual mesh filename=package://centauro_urdf/meshes/v2/ankle-pitch.stl scale=0.001 0.001 0.001
- link ankle2_1: geometry collision cylinder length=0.07370263129636398 radius=0.0813545; visual mesh filename=package://centauro_urdf/meshes/v2/ankle-yaw.stl scale=0.001 -0.001 0.001
- link ankle2_2: geometry collision cylinder length=0.07370263129636398 radius=0.0813545; visual mesh filename=package://centauro_urdf/meshes/v2/ankle-yaw.stl scale=0.001 0.001 0.001
- link ankle2_3: geometry collision cylinder length=0.07370263129636398 radius=0.0813545; visual mesh filename=package://centauro_urdf/meshes/v2/ankle-yaw.stl scale=0.001 -0.001 0.001
- link ankle2_4: geometry collision cylinder length=0.07370263129636398 radius=0.0813545; visual mesh filename=package://centauro_urdf/meshes/v2/ankle-yaw.stl scale=0.001 0.001 0.001
- link arm1_1: geometry collision cylinder length=0.03739768494560427 radius=0.0698859; visual mesh filename=package://centauro_urdf/meshes/ShoulderPitch.STL scale=0.001 -0.001 0.001
- link arm1_2: geometry collision cylinder length=0.12799269981445732 radius=0.0700645; visual mesh filename=package://centauro_urdf/meshes/ShoulderRoll.STL scale=0.001 -0.001 0.001
- link arm1_3: geometry collision cylinder length=0.06082252644344949 radius=0.0896121; visual mesh filename=package://centauro_urdf/meshes/ShoulderYaw.STL scale=0.001 -0.001 0.001
- link arm1_4: geometry collision cylinder length=0.08713418572944408 radius=0.0600429; visual mesh filename=package://centauro_urdf/meshes/Elbow.STL scale=0.001 -0.001 0.001
- link arm1_5: geometry collision cylinder length=0.08434739747702548 radius=0.0804108; visual mesh filename=package://centauro_urdf/meshes/Forearm.STL scale=0.001 -0.001 0.001
- link arm1_6: geometry collision cylinder length=0.11425141871384588 radius=0.0583263; visual mesh filename=package://centauro_urdf/meshes/ForearmPitch.STL scale=0.001 -0.001 0.001
- link arm1_7: geometry collision cylinder length=0.009167307493588288 radius=0.0207073; visual mesh filename=package://centauro_urdf/meshes/ForearmYaw.STL scale=0.001 -0.001 0.001
- link arm1_8: mass 0 -> 0.0
- link arm2_1: geometry collision cylinder length=0.03739768494560427 radius=0.0698859; visual mesh filename=package://centauro_urdf/meshes/ShoulderPitch.STL scale=0.001 0.001 0.001
- link arm2_2: geometry collision cylinder length=0.12799269981445732 radius=0.0700645; visual mesh filename=package://centauro_urdf/meshes/ShoulderRoll.STL scale=0.001 0.001 0.001
- link arm2_3: geometry collision cylinder length=0.06082252644344949 radius=0.0896121; visual mesh filename=package://centauro_urdf/meshes/ShoulderYaw.STL scale=0.001 0.001 0.001
- link arm2_4: geometry collision cylinder length=0.08713418572944408 radius=0.0600429; visual mesh filename=package://centauro_urdf/meshes/Elbow.STL scale=0.001 0.001 0.001
- link arm2_5: geometry collision cylinder length=0.08434739747702548 radius=0.0804108; visual mesh filename=package://centauro_urdf/meshes/Forearm.STL scale=0.001 0.001 0.001
- link arm2_6: geometry collision cylinder length=0.11425141871384588 radius=0.0583263; visual mesh filename=package://centauro_urdf/meshes/ForearmPitch.STL scale=0.001 0.001 0.001
- link arm2_7: geometry collision cylinder length=0.009167307493588288 radius=0.0207073; visual mesh filename=package://centauro_urdf/meshes/ForearmYaw.STL scale=0.001 0.001 0.001
- link arm2_8: mass 0 -> 0.0
- link ball1: geometry collision cylinder length=9.940076835940455e-05 radius=0.0709883; visual mesh filename=package://centauro_urdf/meshes/BallHand.stl scale=0.001 0.001 0.001
- link ball2: geometry collision cylinder length=9.940076835940455e-05 radius=0.0709883; visual mesh filename=package://centauro_urdf/meshes/BallHand.stl scale=0.001 0.001 0.001
- link base_link: geometry collision cylinder length=0.38594139791384763 radius=0.213204; visual mesh filename=package://centauro_urdf/meshes/v2/pelvis.stl scale=0.001 0.001 0.001
- link d435_head_motor: geometry collision cylinder length=0.12134423548428976 radius=0.0261699; visual mesh filename=package://centauro_urdf/meshes/neck-pitch_mesh.stl scale=0.001 0.001 0.001
- link hip1_1: geometry collision cylinder length=0.03069545889898954 radius=0.0747223; visual mesh filename=package://centauro_urdf/meshes/v2/hip-yaw.stl scale=0.001 -0.001 0.001
- link hip1_2: geometry collision cylinder length=0.03069545889898954 radius=0.0747223; visual mesh filename=package://centauro_urdf/meshes/v2/hip-yaw.stl scale=0.001 0.001 0.001
- link hip1_3: geometry collision cylinder length=0.03069545889898954 radius=0.0747223; visual mesh filename=package://centauro_urdf/meshes/v2/hip-yaw.stl scale=0.001 -0.001 0.001
- link hip1_4: geometry collision cylinder length=0.03069545889898954 radius=0.0747223; visual mesh filename=package://centauro_urdf/meshes/v2/hip-yaw.stl scale=0.001 0.001 0.001
- link hip2_1: geometry collision cylinder length=0.2919804521727749 radius=0.0808941; visual mesh filename=package://centauro_urdf/meshes/v2/hip-pitch.stl scale=0.001 0.001 -0.001
- link hip2_2: geometry collision cylinder length=0.2919804521727749 radius=0.0808941; visual mesh filename=package://centauro_urdf/meshes/v2/hip-pitch.stl scale=0.001 0.001 0.001
- link hip2_3: geometry collision cylinder length=0.2919804521727749 radius=0.0808941; visual mesh filename=package://centauro_urdf/meshes/v2/hip-pitch.stl scale=0.001 0.001 -0.001
- link hip2_4: geometry collision cylinder length=0.2919804521727749 radius=0.0808941; visual mesh filename=package://centauro_urdf/meshes/v2/hip-pitch.stl scale=0.001 0.001 0.001
- link knee_1: geometry collision cylinder length=0.19275022460612404 radius=0.0664305; visual mesh filename=package://centauro_urdf/meshes/v2/knee.stl scale=0.001 0.001 -0.001
- link knee_2: geometry collision cylinder length=0.19275022460612404 radius=0.0664305; visual mesh filename=package://centauro_urdf/meshes/v2/knee.stl scale=0.001 0.001 0.001
- link knee_3: geometry collision cylinder length=0.19275022460612404 radius=0.0664305; visual mesh filename=package://centauro_urdf/meshes/v2/knee.stl scale=0.001 0.001 -0.001
- link knee_4: geometry collision cylinder length=0.19275022460612404 radius=0.0664305; visual mesh filename=package://centauro_urdf/meshes/v2/knee.stl scale=0.001 0.001 0.001
- link neck_1: geometry collision cylinder length=0.16454098025546557 radius=0.100414; visual mesh filename=package://centauro_urdf/meshes/head-base_mesh.stl scale=0.001 0.001 0.001
- link torso_2: geometry collision cylinder length=0.09543675990850982 radius=0.158224; visual mesh filename=package://centauro_urdf/meshes/link1_no_head.stl scale=0.001 0.001 0.001
- link velodyne_calib_base_link: geometry collision cylinder length=0.0717 radius=0.0516; visual mesh filename=package://velodyne_description/meshes/VLP16_base_1.dae
- link velodyne_motor: geometry collision cylinder length=0.032463112134515464 radius=0.0544637; visual mesh filename=package://centauro_urdf/meshes/lidar_mesh.stl scale=0.001 0.001 0.001
- link wheel_1: geometry collision cylinder length=0.11 radius=0.078; visual mesh filename=package://centauro_urdf/meshes/v2/wheel.stl scale=0.001 0.001 -0.001
- link wheel_2: geometry collision cylinder length=0.11 radius=0.078; visual mesh filename=package://centauro_urdf/meshes/v2/wheel.stl scale=0.001 0.001 0.001
- link wheel_3: geometry collision cylinder length=0.11 radius=0.078; visual mesh filename=package://centauro_urdf/meshes/v2/wheel.stl scale=0.001 0.001 -0.001
- link wheel_4: geometry collision cylinder length=0.11 radius=0.078; visual mesh filename=package://centauro_urdf/meshes/v2/wheel.stl scale=0.001 0.001 0.001
Joints:
- joint D435_head_camera_accel_joint: origin xyz=-0.00174 0.00552 0.0176 rpy=0 0 0 -> xyz=-0.00174 0.00552 0.0176 rpy=0.0 0.0 0.0
- joint D435_head_camera_accel_optical_joint: origin xyz=0 0 0 rpy=-1.5707963267948966 0 -1.5707963267948966 -> xyz=0.0 0.0 0.0 rpy=-1.5707963267948966 0.0 -1.5707963267948966
- joint D435_head_camera_color_joint: origin xyz=0 0.015 0 rpy=0 0 0 -> xyz=0.0 0.015 0.0 rpy=0.0 0.0 0.0
- joint D435_head_camera_color_optical_joint: origin xyz=0 0 0 rpy=-1.5707963267948966 0 -1.5707963267948966 -> xyz=0.0 0.0 0.0 rpy=-1.5707963267948966 0.0 -1.5707963267948966
- joint D435_head_camera_depth_joint: origin xyz=0 0 0 rpy=0 0 0 -> xyz=0.0 0.0 0.0 rpy=0.0 0.0 0.0
- joint D435_head_camera_depth_optical_joint: origin xyz=0 0 0 rpy=-1.5707963267948966 0 -1.5707963267948966 -> xyz=0.0 0.0 0.0 rpy=-1.5707963267948966 0.0 -1.5707963267948966
- joint D435_head_camera_gyro_joint: origin xyz=-0.00174 0.00552 0.0176 rpy=0 0 0 -> xyz=-0.00174 0.00552 0.0176 rpy=0.0 0.0 0.0
- joint D435_head_camera_gyro_optical_joint: origin xyz=0 0 0 rpy=-1.5707963267948966 0 -1.5707963267948966 -> xyz=0.0 0.0 0.0 rpy=-1.5707963267948966 0.0 -1.5707963267948966
- joint D435_head_camera_joint: origin xyz=0.03015 0 -0.0125 rpy=0 0 0 -> xyz=0.03015 0.0 -0.0125 rpy=0.0 0.0 0.0
- joint D435_head_camera_left_ir_joint: origin xyz=0 0.0 0 rpy=0 0 0 -> xyz=0.0 0.0 0.0 rpy=0.0 0.0 0.0
- joint D435_head_camera_left_ir_optical_joint: origin xyz=0 0 0 rpy=-1.5707963267948966 0 -1.5707963267948966 -> xyz=0.0 0.0 0.0 rpy=-1.5707963267948966 0.0 -1.5707963267948966
- joint D435_head_camera_link_joint: origin xyz=0 0.0175 0.0125 rpy=0 0 0 -> xyz=0.0 0.0175 0.0125 rpy=0.0 0.0 0.0
- joint D435_head_camera_right_ir_joint: origin xyz=0 -0.05 0 rpy=0 0 0 -> xyz=0.0 -0.05 0.0 rpy=0.0 0.0 0.0
- joint D435_head_camera_right_ir_optical_joint: origin xyz=0 0 0 rpy=-1.5707963267948966 0 -1.5707963267948966 -> xyz=0.0 0.0 0.0 rpy=-1.5707963267948966 0.0 -1.5707963267948966
- joint D435i_camera_accel_joint: origin xyz=-0.00174 0.00552 0.0176 rpy=0 0 0 -> xyz=-0.00174 0.00552 0.0176 rpy=0.0 0.0 0.0
- joint D435i_camera_accel_optical_joint: origin xyz=0 0 0 rpy=-1.5707963267948966 0 -1.5707963267948966 -> xyz=0.0 0.0 0.0 rpy=-1.5707963267948966 0.0 -1.5707963267948966
- joint D435i_camera_color_joint: origin xyz=0 0.015 0 rpy=0 0 0 -> xyz=0.0 0.015 0.0 rpy=0.0 0.0 0.0
- joint D435i_camera_color_optical_joint: origin xyz=0 0 0 rpy=-1.5707963267948966 0 -1.5707963267948966 -> xyz=0.0 0.0 0.0 rpy=-1.5707963267948966 0.0 -1.5707963267948966
- joint D435i_camera_depth_joint: origin xyz=0 0 0 rpy=0 0 0 -> xyz=0.0 0.0 0.0 rpy=0.0 0.0 0.0
- joint D435i_camera_depth_optical_joint: origin xyz=0 0 0 rpy=-1.5707963267948966 0 -1.5707963267948966 -> xyz=0.0 0.0 0.0 rpy=-1.5707963267948966 0.0 -1.5707963267948966
- joint D435i_camera_gyro_joint: origin xyz=-0.00174 0.00552 0.0176 rpy=0 0 0 -> xyz=-0.00174 0.00552 0.0176 rpy=0.0 0.0 0.0
- joint D435i_camera_gyro_optical_joint: origin xyz=0 0 0 rpy=-1.5707963267948966 0 -1.5707963267948966 -> xyz=0.0 0.0 0.0 rpy=-1.5707963267948966 0.0 -1.5707963267948966
- joint D435i_camera_joint: origin xyz=0.27187 0 0.0215997 rpy=0 0.5251508 0 -> xyz=0.27187 0.0 0.0215997 rpy=0.0 0.5251508 0.0
- joint D435i_camera_left_ir_joint: origin xyz=0 0.0 0 rpy=0 0 0 -> xyz=0.0 0.0 0.0 rpy=0.0 0.0 0.0
- joint D435i_camera_left_ir_optical_joint: origin xyz=0 0 0 rpy=-1.5707963267948966 0 -1.5707963267948966 -> xyz=0.0 0.0 0.0 rpy=-1.5707963267948966 0.0 -1.5707963267948966
- joint D435i_camera_link_joint: origin xyz=0 0.0175 0.0125 rpy=0 0 0 -> xyz=0.0 0.0175 0.0125 rpy=0.0 0.0 0.0
- joint D435i_camera_right_ir_joint: origin xyz=0 -0.05 0 rpy=0 0 0 -> xyz=0.0 -0.05 0.0 rpy=0.0 0.0 0.0
- joint D435i_camera_right_ir_optical_joint: origin xyz=0 0 0 rpy=-1.5707963267948966 0 -1.5707963267948966 -> xyz=0.0 0.0 0.0 rpy=-1.5707963267948966 0.0 -1.5707963267948966
- joint T265_camera_accel_joint: origin xyz=-0.0311 0 0.00655 rpy=0 3.141592653589793 0 -> xyz=-0.0311 0.0 0.00655 rpy=0.0 3.141592653589793 0.0
- joint T265_camera_accel_optical_joint: origin xyz=-0.0311 0 0.00655 rpy=0 3.141592653589793 0 -> xyz=-0.0311 0.0 0.00655 rpy=0.0 3.141592653589793 0.0
- joint T265_camera_fisheye1_optical_joint: origin xyz=0 0 0 rpy=-1.5707963267948966 0 -1.5707963267948966 -> xyz=0.0 0.0 0.0 rpy=-1.5707963267948966 0.0 -1.5707963267948966
- joint T265_camera_fisheye1_rgb_joint: origin xyz=-0.0411 0.0 0.0 rpy=0 1.5707963267948966 1.5707963267948966 -> xyz=-0.0411 0.0 0.0 rpy=0.0 1.5707963267948966 1.5707963267948966
- joint T265_camera_fisheye2_optical_joint: origin xyz=0 0 0 rpy=-1.5707963267948966 0 -1.5707963267948966 -> xyz=0.0 0.0 0.0 rpy=-1.5707963267948966 0.0 -1.5707963267948966
- joint T265_camera_fisheye2_rgb_joint: origin xyz=0.0229 0.0 0.0 rpy=0 1.5707963267948966 1.5707963267948966 -> xyz=0.0229 0.0 0.0 rpy=0.0 1.5707963267948966 1.5707963267948966
- joint T265_camera_gyro_joint: origin xyz=-0.0311 0 0.00655 rpy=0 3.141592653589793 0 -> xyz=-0.0311 0.0 0.00655 rpy=0.0 3.141592653589793 0.0
- joint T265_camera_gyro_optical_joint: origin xyz=0 0 0 rpy=0 0 0 -> xyz=0.0 0.0 0.0 rpy=0.0 0.0 0.0
- joint T265_camera_link_joint: origin xyz=0 0 0 rpy=1.5707963267948966 0 -1.5707963267948966 -> xyz=0.0 0.0 0.0 rpy=1.5707963267948966 0.0 -1.5707963267948966
- joint T265_camera_pose_joint: origin xyz=0.29245 0.00775 0.063 rpy=0 0 0 -> xyz=0.29245 0.00775 0.063 rpy=0.0 0.0 0.0
- joint ankle_pitch_1: axis 0 0 -1 -> 0.0 0.0 -1.0; limit lower=-2.4056 upper=2.3184 effort=147 velocity=8.1 -> lower=-2.4056 upper=2.3184 effort=147.0 velocity=8.1
- joint ankle_pitch_2: axis 0 0 1 -> 0.0 0.0 1.0; limit lower=-2.3266 upper=2.3914 effort=147 velocity=8.1 -> lower=-2.3266 upper=2.3914 effort=147.0 velocity=8.1
- joint ankle_pitch_3: axis 0 0 -1 -> 0.0 0.0 -1.0; limit lower=-2.4696 upper=2.4464 effort=147 velocity=8.1 -> lower=-2.4696 upper=2.4464 effort=147.0 velocity=8.1
- joint ankle_pitch_4: axis 0 0 1 -> 0.0 0.0 1.0; limit lower=-2.3426 upper=2.3934 effort=147 velocity=8.1 -> lower=-2.3426 upper=2.3934 effort=147.0 velocity=8.1
- joint ankle_yaw_1: axis 0 0 -1 -> 0.0 0.0 -1.0; limit lower=-2.5626 upper=2.5384 effort=35 velocity=20.0 -> lower=-2.5626 upper=2.5384 effort=35.0 velocity=20.0
- joint ankle_yaw_2: axis 0 0 -1 -> 0.0 0.0 -1.0; limit lower=-2.5546 upper=2.5484 effort=35 velocity=20.0 -> lower=-2.5546 upper=2.5484 effort=35.0 velocity=20.0
- joint ankle_yaw_3: axis 0 0 -1 -> 0.0 0.0 -1.0; limit lower=-2.5606 upper=2.5454 effort=35 velocity=20.0 -> lower=-2.5606 upper=2.5454 effort=35.0 velocity=20.0
- joint ankle_yaw_4: axis 0 0 -1 -> 0.0 0.0 -1.0; limit lower=-2.6046 upper=2.5514 effort=35 velocity=20.0 -> lower=-2.6046 upper=2.5514 effort=35.0 velocity=20.0
- joint base_to_base_inertia: origin xyz=0 0 0 rpy=0 0 0 -> xyz=0.0 0.0 0.0 rpy=0.0 0.0 0.0
- joint contact_joint_1: origin xyz=0 0 -0.176 rpy=0 0 0 -> xyz=0.0 0.0 -0.176 rpy=0.0 0.0 0.0
- joint contact_joint_2: origin xyz=0 0 -0.176 rpy=0 0 0 -> xyz=0.0 0.0 -0.176 rpy=0.0 0.0 0.0
- joint contact_joint_3: origin xyz=0 0 -0.176 rpy=0 0 0 -> xyz=0.0 0.0 -0.176 rpy=0.0 0.0 0.0
- joint contact_joint_4: origin xyz=0 0 -0.176 rpy=0 0 0 -> xyz=0.0 0.0 -0.176 rpy=0.0 0.0 0.0
- joint d435_head_joint: origin xyz=0.06 0 0.1375 rpy=0 0 0 -> xyz=0.06 0.0 0.1375 rpy=0.0 0.0 0.0
- joint hip_pitch_1: axis 0 0 -1 -> 0.0 0.0 -1.0; limit lower=-2.0226 upper=2.02748 effort=304 velocity=8.8 -> lower=-2.0226 upper=2.02748 effort=304.0 velocity=8.8
- joint hip_pitch_2: axis 0 0 1 -> 0.0 0.0 1.0; limit lower=-2.0156 upper=2.0354 effort=304 velocity=8.8 -> lower=-2.0156 upper=2.0354 effort=304.0 velocity=8.8
- joint hip_pitch_3: axis 0 0 -1 -> 0.0 0.0 -1.0; limit lower=-2.0126 upper=2.0384 effort=304 velocity=8.8 -> lower=-2.0126 upper=2.0384 effort=304.0 velocity=8.8
- joint hip_pitch_4: axis 0 0 1 -> 0.0 0.0 1.0; limit lower=-2.0326 upper=2.0524 effort=304 velocity=8.8 -> lower=-2.0326 upper=2.0524 effort=304.0 velocity=8.8
- joint hip_yaw_1: axis 0 0 -1 -> 0.0 0.0 -1.0; limit lower=-2.03 upper=2.51 effort=304 velocity=8.8 -> lower=-2.03 upper=2.51 effort=304.0 velocity=8.8
- joint hip_yaw_2: axis 0 0 -1 -> 0.0 0.0 -1.0; limit lower=-2.51 upper=2.03 effort=304 velocity=8.8 -> lower=-2.51 upper=2.03 effort=304.0 velocity=8.8
- joint hip_yaw_3: axis 0 0 -1 -> 0.0 0.0 -1.0; limit lower=-2.51 upper=2.03 effort=304 velocity=8.8 -> lower=-2.51 upper=2.03 effort=304.0 velocity=8.8
- joint hip_yaw_4: axis 0 0 -1 -> 0.0 0.0 -1.0; limit lower=-2.03 upper=2.51 effort=304 velocity=8.8 -> lower=-2.03 upper=2.51 effort=304.0 velocity=8.8
- joint j_arm1_1: axis 0 1 0 -> 0.0 1.0 0.0
- joint j_arm1_2: axis 1 0 0 -> 1.0 0.0 0.0
- joint j_arm1_3: axis 0 0 1 -> 0.0 0.0 1.0; origin xyz=0.09015 0.0 -0.21815 -> xyz=0.09015 0.0 -0.21815 rpy=0.0 0.0 0.0
- joint j_arm1_4: axis 0 1 0 -> 0.0 1.0 0.0; origin xyz=0.045 0.05515 -0.074 -> xyz=0.045 0.05515 -0.074 rpy=0.0 0.0 0.0
- joint j_arm1_5: axis 0 0 1 -> 0.0 0.0 1.0; origin xyz=-0.015 -0.05515 -0.095 -> xyz=-0.015 -0.05515 -0.095 rpy=0.0 0.0 0.0
- joint j_arm1_6: axis 0 1 0 -> 0.0 1.0 0.0; origin xyz=0.0 0.049 -0.156 -> xyz=0.0 0.049 -0.156 rpy=0.0 0.0 0.0
- joint j_arm1_7: axis 0 0 1 -> 0.0 0.0 1.0; origin xyz=0.0 -0.049 -0.174 -> xyz=0.0 -0.049 -0.174 rpy=0.0 0.0 0.0
- joint j_arm1_8: origin xyz=0. 0. 0. rpy=0. 0. 0. -> xyz=0.0 0.0 0.0 rpy=0.0 0.0 0.0
- joint j_arm2_1: axis 0 1 0 -> 0.0 1.0 0.0
- joint j_arm2_2: axis 1 0 0 -> 1.0 0.0 0.0
- joint j_arm2_3: axis 0 0 1 -> 0.0 0.0 1.0; origin xyz=0.09015 0.0 -0.21815 -> xyz=0.09015 0.0 -0.21815 rpy=0.0 0.0 0.0
- joint j_arm2_4: axis 0 1 0 -> 0.0 1.0 0.0; origin xyz=0.045 -0.05515 -0.074 -> xyz=0.045 -0.05515 -0.074 rpy=0.0 0.0 0.0
- joint j_arm2_5: axis 0 0 1 -> 0.0 0.0 1.0; origin xyz=-0.015 0.05515 -0.095 -> xyz=-0.015 0.05515 -0.095 rpy=0.0 0.0 0.0
- joint j_arm2_6: axis 0 1 0 -> 0.0 1.0 0.0; origin xyz=0.0 -0.049 -0.156 -> xyz=0.0 -0.049 -0.156 rpy=0.0 0.0 0.0
- joint j_arm2_7: axis 0 0 1 -> 0.0 0.0 1.0; origin xyz=0.0 0.049 -0.174 -> xyz=0.0 0.049 -0.174 rpy=0.0 0.0 0.0
- joint j_arm2_8: origin xyz=0. 0. 0. rpy=0. 0. 0. -> xyz=0.0 0.0 0.0 rpy=0.0 0.0 0.0
- joint j_ball1_tip: origin xyz=0 0 -0.07 rpy=0 0 0 -> xyz=0.0 0.0 -0.07 rpy=0.0 0.0 0.0
- joint j_ball2_tip: origin xyz=0 0 -0.07 rpy=0 0 0 -> xyz=0.0 0.0 -0.07 rpy=0.0 0.0 0.0
- joint j_ft_1: axis 0 0 1 -> 0.0 0.0 1.0; limit lower=0.0 upper=0.0 effort=0 velocity=0 -> lower=0.0 upper=0.0 effort=0.0 velocity=0.0
- joint j_ft_2: axis 0 0 1 -> 0.0 0.0 1.0; limit lower=0.0 upper=0.0 effort=0 velocity=0 -> lower=0.0 upper=0.0 effort=0.0 velocity=0.0
- joint j_wheel_1: axis 0 0 -1 -> 0.0 0.0 -1.0; limit lower=-62.83 upper=62.83 effort=35 velocity=20.0 -> lower=-62.83 upper=62.83 effort=35.0 velocity=20.0
- joint j_wheel_2: axis 0 0 1 -> 0.0 0.0 1.0; limit lower=-62.83 upper=62.83 effort=35 velocity=20.0 -> lower=-62.83 upper=62.83 effort=35.0 velocity=20.0
- joint j_wheel_3: axis 0 0 -1 -> 0.0 0.0 -1.0; limit lower=-62.83 upper=62.83 effort=35 velocity=20.0 -> lower=-62.83 upper=62.83 effort=35.0 velocity=20.0
- joint j_wheel_4: axis 0 0 1 -> 0.0 0.0 1.0; limit lower=-62.83 upper=62.83 effort=35 velocity=20.0 -> lower=-62.83 upper=62.83 effort=35.0 velocity=20.0
- joint knee_pitch_1: axis 0 0 -1 -> 0.0 0.0 -1.0; limit lower=-2.4056 upper=2.3994 effort=304 velocity=8.8 -> lower=-2.4056 upper=2.3994 effort=304.0 velocity=8.8
- joint knee_pitch_2: axis 0 0 1 -> 0.0 0.0 1.0; limit lower=-2.4006 upper=2.4034 effort=304 velocity=8.8 -> lower=-2.4006 upper=2.4034 effort=304.0 velocity=8.8
- joint knee_pitch_3: axis 0 0 -1 -> 0.0 0.0 -1.0; limit lower=-2.4056 upper=2.4064 effort=304 velocity=8.8 -> lower=-2.4056 upper=2.4064 effort=304.0 velocity=8.8
- joint knee_pitch_4: axis 0 0 1 -> 0.0 0.0 1.0; limit lower=-2.4176 upper=2.3884 effort=304 velocity=8.8 -> lower=-2.4176 upper=2.3884 effort=304.0 velocity=8.8
- joint neck_base: axis 0 0 1 -> 0.0 0.0 1.0; origin xyz=0.0030637045 0.0061607221 0.158 rpy=0 0 0 -> xyz=0.0030637045 0.0061607221 0.158 rpy=0.0 0.0 0.0
- joint torso_yaw: axis 0 0 1 -> 0.0 0.0 1.0; limit lower=-2.618 upper=2.618 effort=147 velocity=5.7 -> lower=-2.618 upper=2.618 effort=147.0 velocity=5.7; origin xyz=0.2 0.0 0.256 -> xyz=0.2 0.0 0.256 rpy=0.0 0.0 0.0
- joint velodyne_calib_base_mount_joint: origin xyz=0 0 0 rpy=0 0 0 -> xyz=0.0 0.0 0.0 rpy=0.0 0.0 0.0
- joint velodyne_calib_base_scan_joint: origin xyz=0 0 0.0377 rpy=0 0 0 -> xyz=0.0 0.0 0.0377 rpy=0.0 0.0 0.0
- joint velodyne_joint: origin xyz=0.0822724 0 0.242 rpy=0 0 0 -> xyz=0.0822724 0.0 0.242 rpy=0.0 0.0 0.0

Commit message: remove wrist joint

File: resources/centauro/urdf/centauro_horizon.urdf (robot description, URDF)
Before this commit: robot centauro, 97 links, 96 joints
Links:
- removed link arm1_7
- removed link arm2_7
- removed link ft_arm1
- removed link ft_arm2
- link arm1_6: geometry collision cylinder length=0.07750977987441161 radius=0.0474698; visual mesh filename=package://centauro_urdf/meshes/wrist_pitch_right.stl scale=0.001 -0.001 0.001
- link arm2_6: geometry collision cylinder length=0.07750977987441161 radius=0.0474698; visual mesh filename=package://centauro_urdf/meshes/wrist_pitch_right.stl scale=0.001 0.001 0.001
Joints:
- removed joint j_arm1_7
- removed joint j_arm2_7
- removed joint j_ft_1
- removed joint j_ft_2
- joint j_arm1_8: origin xyz=0.0 0.0 0.0 rpy=0.0 0.0 0.0 -> xyz=0.0 -0.05 -0.105 rpy=0.0 0.0 0.0; parent arm1_7 -> arm1_6
- joint j_arm2_8: origin xyz=0.0 0.0 0.0 rpy=0.0 0.0 0.0 -> xyz=0.0 0.05 -0.105 rpy=0.0 0.0 0.0; parent arm2_7 -> arm2_6
