Commit message: add tcp frame

File: resources/centauro/urdf/centauro_dagana.urdf (robot description, URDF)
Before this commit: robot centauro, 93 links, 92 joints
Links:
- added link dagana_2_tcp
Joints:
- added joint dagana_2_tcp_joint: type fixed, parent dagana_2_top_link, child dagana_2_tcp, origin xyz=0 -0.05 0.15 rpy=0 0 0

Commit message: arm2_8 whould have dagana bottom link as parent

File: resources/centauro/urdf/centauro_dagana.urdf (robot description, URDF)
Before this commit: robot centauro, 94 links, 93 joints
Joints:
- joint j_arm2_8: parent dagana_2_top_link -> dagana_2_bottom_link

Commit message: add big wheels

File: resources/centauro/urdf/centauro_dagana.urdf (robot description, URDF)
Before this commit: robot centauro, 94 links, 93 joints
Links:
- link ankle2_1: mass 1.7656714 -> 2.440929; geometry collision cylinder length=0.13078435048455633 radius=0.08586; visual mesh filename=package://centauro_urdf/meshes/v2/mesh_ankle-yaw_wheel23.stl scale=0.001 -0.001 0.001
- link ankle2_2: mass 1.7656714 -> 2.440929; geometry collision cylinder length=0.13078435048455633 radius=0.08586; visual mesh filename=package://centauro_urdf/meshes/v2/mesh_ankle-yaw_wheel23.stl scale=0.001 0.001 0.001
- link ankle2_3: mass 1.7656714 -> 2.440929; geometry collision cylinder length=0.13078435048455633 radius=0.08586; visual mesh filename=package://centauro_urdf/meshes/v2/mesh_ankle-yaw_wheel23.stl scale=0.001 -0.001 0.001
- link ankle2_4: mass 1.7656714 -> 2.440929; geometry collision cylinder length=0.13078435048455633 radius=0.08586; visual mesh filename=package://centauro_urdf/meshes/v2/mesh_ankle-yaw_wheel23.stl scale=0.001 0.001 0.001
- link wheel_1: mass 1.11164 -> 1.8569388; geometry collision cylinder length=0.0004424382093719415 radius=0.119659; visual mesh filename=package://centauro_urdf/meshes/v2/mesh_wheel23.stl scale=0.001 0.001 -0.001
- link wheel_2: mass 1.11164 -> 1.8569388; geometry collision cylinder length=0.0004424382093719415 radius=0.119659; visual mesh filename=package://centauro_urdf/meshes/v2/mesh_wheel23.stl scale=0.001 0.001 0.001
- link wheel_3: mass 1.11164 -> 1.8569388; geometry collision cylinder length=0.0004424382093719415 radius=0.119659; visual mesh filename=package://centauro_urdf/meshes/v2/mesh_wheel23.stl scale=0.001 0.001 -0.001
- link wheel_4: mass 1.11164 -> 1.8569388; geometry collision cylinder length=0.0004424382093719415 radius=0.119659; visual mesh filename=package://centauro_urdf/meshes/v2/mesh_wheel23.stl scale=0.001 0.001 0.001
Joints:
- joint contact_joint_1: origin xyz=0.0 0.0 -0.176 rpy=0.0 0.0 0.0 -> xyz=0 0 -0.26835 rpy=0 0 0
- joint contact_joint_2: origin xyz=0.0 0.0 -0.176 rpy=0.0 0.0 0.0 -> xyz=0 0 -0.26835 rpy=0 0 0
- joint contact_joint_3: origin xyz=0.0 0.0 -0.176 rpy=0.0 0.0 0.0 -> xyz=0 0 -0.26835 rpy=0 0 0
- joint contact_joint_4: origin xyz=0.0 0.0 -0.176 rpy=0.0 0.0 0.0 -> xyz=0 0 -0.26835 rpy=0 0 0
- joint dagana_2_mount_joint: origin xyz=0.0 0.05 -0.08 rpy=0.0 3.14159265359 3.14159265359 -> xyz=0.0 0.05 -0.08 rpy=0.0 3.14159265359 0
- joint j_wheel_1: axis 0.0 0.0 -1.0 -> 0 0 -1; limit lower=-62.83 upper=62.83 effort=35.0 velocity=20.0 -> lower=-62.83 upper=62.83 effort=35 velocity=20.0; origin xyz=0.0 -0.0 -0.09834999999999999 rpy=1.57079632679 0.0 0.0 -> xyz=0.0 -0.0 -0.14435 rpy=1.57079632679 0.0 0.0
- joint j_wheel_2: axis 0.0 0.0 1.0 -> 0 0 1; limit lower=-62.83 upper=62.83 effort=35.0 velocity=20.0 -> lower=-62.83 upper=62.83 effort=35 velocity=20.0; origin xyz=0.0 0.0 -0.09834999999999999 rpy=1.57079632679 0.0 0.0 -> xyz=0.0 0.0 -0.14435 rpy=1.57079632679 0.0 0.0
- joint j_wheel_3: axis 0.0 0.0 -1.0 -> 0 0 -1; limit lower=-62.83 upper=62.83 effort=35.0 velocity=20.0 -> lower=-62.83 upper=62.83 effort=35 velocity=20.0; origin xyz=0.0 -0.0 -0.09834999999999999 rpy=1.57079632679 0.0 0.0 -> xyz=0.0 -0.0 -0.14435 rpy=1.57079632679 0.0 0.0
- joint j_wheel_4: axis 0.0 0.0 1.0 -> 0 0 1; limit lower=-62.83 upper=62.83 effort=35.0 velocity=20.0 -> lower=-62.83 upper=62.83 effort=35 velocity=20.0; origin xyz=0.0 0.0 -0.09834999999999999 rpy=1.57079632679 0.0 0.0 -> xyz=0.0 0.0 -0.14435 rpy=1.57079632679 0.0 0.0

File: resources/centauro/urdf/centauro_horizon.urdf (robot description, URDF)
Before this commit: robot centauro, 93 links, 92 joints
Links:
- link ankle2_1: mass 1.7656714 -> 2.440929; geometry collision cylinder length=0.13078435048455633 radius=0.08586; visual mesh filename=package://centauro_urdf/meshes/v2/mesh_ankle-yaw_wheel23.stl scale=0.001 -0.001 0.001
- link ankle2_2: mass 1.7656714 -> 2.440929; geometry collision cylinder length=0.13078435048455633 radius=0.08586; visual mesh filename=package://centauro_urdf/meshes/v2/mesh_ankle-yaw_wheel23.stl scale=0.001 0.001 0.001
- link ankle2_3: mass 1.7656714 -> 2.440929; geometry collision cylinder length=0.13078435048455633 radius=0.08586; visual mesh filename=package://centauro_urdf/meshes/v2/mesh_ankle-yaw_wheel23.stl scale=0.001 -0.001 0.001
- link ankle2_4: mass 1.7656714 -> 2.440929; geometry collision cylinder length=0.13078435048455633 radius=0.08586; visual mesh filename=package://centauro_urdf/meshes/v2/mesh_ankle-yaw_wheel23.stl scale=0.001 0.001 0.001
- link wheel_1: mass 1.11164 -> 1.8569388; geometry collision cylinder length=0.0004424382093719415 radius=0.119659; visual mesh filename=package://centauro_urdf/meshes/v2/mesh_wheel23.stl scale=0.001 0.001 -0.001
- link wheel_2: mass 1.11164 -> 1.8569388; geometry collision cylinder length=0.0004424382093719415 radius=0.119659; visual mesh filename=package://centauro_urdf/meshes/v2/mesh_wheel23.stl scale=0.001 0.001 0.001
- link wheel_3: mass 1.11164 -> 1.8569388; geometry collision cylinder length=0.0004424382093719415 radius=0.119659; visual mesh filename=package://centauro_urdf/meshes/v2/mesh_wheel23.stl scale=0.001 0.001 -0.001
- link wheel_4: mass 1.11164 -> 1.8569388; geometry collision cylinder length=0.0004424382093719415 radius=0.119659; visual mesh filename=package://centauro_urdf/meshes/v2/mesh_wheel23.stl scale=0.001 0.001 0.001
Joints:
- joint contact_joint_1: origin xyz=0.0 0.0 -0.176 rpy=0.0 0.0 0.0 -> xyz=0 0 -0.26835 rpy=0 0 0
- joint contact_joint_2: origin xyz=0.0 0.0 -0.176 rpy=0.0 0.0 0.0 -> xyz=0 0 -0.26835 rpy=0 0 0
- joint contact_joint_3: origin xyz=0.0 0.0 -0.176 rpy=0.0 0.0 0.0 -> xyz=0 0 -0.26835 rpy=0 0 0
- joint contact_joint_4: origin xyz=0.0 0.0 -0.176 rpy=0.0 0.0 0.0 -> xyz=0 0 -0.26835 rpy=0 0 0
- joint j_wheel_1: axis 0.0 0.0 -1.0 -> 0 0 -1; limit lower=-62.83 upper=62.83 effort=35.0 velocity=20.0 -> lower=-62.83 upper=62.83 effort=35 velocity=20.0; origin xyz=0.0 -0.0 -0.09834999999999999 rpy=1.57079632679 0.0 0.0 -> xyz=0.0 -0.0 -0.14435 rpy=1.57079632679 0.0 0.0
- joint j_wheel_2: axis 0.0 0.0 1.0 -> 0 0 1; limit lower=-62.83 upper=62.83 effort=35.0 velocity=20.0 -> lower=-62.83 upper=62.83 effort=35 velocity=20.0; origin xyz=0.0 0.0 -0.09834999999999999 rpy=1.57079632679 0.0 0.0 -> xyz=0.0 0.0 -0.14435 rpy=1.57079632679 0.0 0.0
- joint j_wheel_3: axis 0.0 0.0 -1.0 -> 0 0 -1; limit lower=-62.83 upper=62.83 effort=35.0 velocity=20.0 -> lower=-62.83 upper=62.83 effort=35 velocity=20.0; origin xyz=0.0 -0.0 -0.09834999999999999 rpy=1.57079632679 0.0 0.0 -> xyz=0.0 -0.0 -0.14435 rpy=1.57079632679 0.0 0.0
- joint j_wheel_4: axis 0.0 0.0 1.0 -> 0 0 1; limit lower=-62.83 upper=62.83 effort=35.0 velocity=20.0 -> lower=-62.83 upper=62.83 effort=35 velocity=20.0; origin xyz=0.0 0.0 -0.09834999999999999 rpy=1.57079632679 0.0 0.0 -> xyz=0.0 0.0 -0.14435 rpy=1.57079632679 0.0 0.0
